File: laser_buck_driver.sch (EAGLE design)
At the start: 23 parts, among them IC1 LM358D, IC2 LM2576, SW1 TACT

Commit message: comments
screenshot and minor updates
Parts:
- R10: value 100k -> 470k
- R4, R5: value 22k -> 100k
Other:
- note added: "470-> 0..2.6A max"
- note added: "bylo 100k"
Changed lines of the file:
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@@
 <part name="C2" library="rcl" deviceset="CPOL-EU" device="153CLV-0810" value="100u/25V"/>
 <part name="R3" library="rcl" deviceset="R-EU_" device="R1206" value="0.1R"/>
-<part name="R4" library="rcl" deviceset="R-EU_" device="R0805" value="22k"/>
-<part name="R5" library="rcl" deviceset="R-EU_" device="R0805" value="22k"/>
+<part name="R4" library="rcl" deviceset="R-EU_" device="R0805" value="100k"/>
+<part name="R5" library="rcl" deviceset="R-EU_" device="R0805" value="100k"/>
 <part name="R6" library="rcl" deviceset="R-EU_" device="R0805" value="100k"/>
 <part name="R7" library="rcl" deviceset="R-EU_" device="R0805" value="100k"/>
 <part name="R8" library="rcl" deviceset="R-EU_" device="R0805" value="20k/do_pominiecia"/>
 <part name="R9" library="rcl" deviceset="R-EU_" device="R0805" value="1k"/>
-<part name="R10" library="rcl" deviceset="R-EU_" device="R0805" value="100k"/>
+<part name="R10" library="rcl" deviceset="R-EU_" device="R0805" value="470k"/>
 <part name="GND1" library="supply1" deviceset="GND" device=""/>
 <part name="GND2" library="supply1" deviceset="GND" device=""/>
@@
 <sheet>
 <plain>
+<text x="127" y="-15.24" size="1.27" layer="91">bylo 100k</text>
+<text x="127" y="-17.78" size="1.27" layer="91">470-&gt; 0..2.6A max</text>
 </plain>
 <instances>
